Commit message: Update base.urdf.xacro

File: race2_description/urdf/base.urdf.xacro (robot description, xacro)
@@ -51,11 +51,4 @@
         <child link="pressure"/>
     </joint>
-    <!-- thrusters -->
-    <!-- <link name="surge_thruster_link"/>
-    <joint name="surge_thruster_joint" type="fixed">
-        <origin xyz="-0.68 0.0 0.0" rpy="0.0 0.0 0.0"/>
-        <parent link="base_link"/>
-        <child link="surge_thruster_link"/>
-    </joint> -->
     <link name="surge_port_thruster_link"/>
     <joint name="race2/surge_port_servo_joint" type="revolute">
@@ -74,17 +67,4 @@
         <limit effort="10" lower="-1.57" upper="1.57" velocity="10"/>
     </joint>
-    <!-- new front-facing thrusters -->
-    <!-- <link name="front_left_thruster_link"/>
-    <joint name="front_left_thruster_joint" type="continuous">
-        <origin xyz="0.0 0.1 0.0" rpy="0.0 0.0 0.0"/>
-        <parent link="base_link"/>
-        <child link="front_left_thruster_link"/>
-    </joint>
-    <link name="front_right_thruster_link"/>
-    <joint name="front_right_thruster_joint" type="continuous">
-        <origin xyz="0.0 -0.1 0.0" rpy="0.0 0.0 0.0"/>
-        <parent link="base_link"/>
-        <child link="front_right_thruster_link"/>
-    </joint> -->
     <!-- Heave Bow Thruster -->
     <link name="heave_bow_thruster_link"/>

Commit message: Control fix

File: race2_description/urdf/base.urdf.xacro (robot description, xacro)
@@ -75,16 +75,16 @@
     </joint>
     <!-- Heave Stern Thruster Port -->
-    <link name="heave_stern_thruster_port_link"/>
-    <joint name="heave_stern_thruster_port_joint" type="fixed">
+    <link name="heave_stern_port_thruster_link"/>
+    <joint name="heave_stern_port_thruster_joint" type="fixed">
         <origin xyz="-0.56 -0.1034 -0.07535" rpy="0.0 1.57079632679 0.0"/>
         <parent link="base_link"/>
-        <child link="heave_stern_thruster_port_link"/>
+        <child link="heave_stern_port_thruster_link"/>
     </joint>
     <!-- Heave Stern Thruster Stbd -->
-    <link name="heave_stern_thruster_stbd_link"/>
-    <joint name="heave_stern_thruster_stbd_joint" type="fixed">
+    <link name="heave_stern_stbd_thruster_link"/>
+    <joint name="heave_stern_stbd_thruster_joint" type="fixed">
         <origin xyz="-0.56 0.1034 -0.07535" rpy="0.0 1.57079632679 0.0"/>
         <parent link="base_link"/>
-        <child link="heave_stern_thruster_stbd_link"/>
+        <child link="heave_stern_stbd_thruster_link"/>
     </joint>
     <!-- Sway Stern Thruster -->

Commit message: Return to standard namespace and joint correction

File: race2_description/urdf/base.urdf.xacro (robot description, xacro)
@@ -51,20 +51,24 @@
         <child link="pressure"/>
     </joint>
-    <link name="surge_port_thruster_link"/>
+    <!-- Start: Port Surge -->
+    <link name="surge_port_duct_link"/>
     <joint name="race2/surge_port_servo_joint" type="revolute">
         <origin xyz="-0.86 -0.125 -0.05485" rpy="-1.5707 0.0 -0.52"/>
         <parent link="base_link"/>
-        <child link="surge_port_thruster_link"/>
+        <child link="surge_port_duct_link"/>
         <axis xyz="0 0 1"/>
         <limit effort="10" lower="-1.57" upper="1.57" velocity="10"/>
     </joint>
-    <link name="surge_starboard_thruster_link"/>
+    <!-- End: Port Surge -->
+    <!-- Start: Starboard Surge -->
+    <link name="surge_starbrd_duct_link"/>
     <joint name="race2/surge_starboard_servo_joint" type="revolute">
         <origin xyz="-0.86 0.125 -0.05485" rpy="1.5707 0.0 0.52"/>
         <parent link="base_link"/>
-        <child link="surge_starboard_thruster_link"/>
+        <child link="surge_starbrd_duct_link"/>
         <axis xyz="0 0 1"/>
         <limit effort="10" lower="-1.57" upper="1.57" velocity="10"/>
     </joint>
+    <!-- End: Starboard Surge -->
     <!-- Heave Bow Thruster -->
     <link name="heave_bow_thruster_link"/>

Commit message: Surge Port Addition!

File: race2_description/urdf/base.urdf.xacro (robot description, xacro)
@@ -52,27 +52,50 @@
     </joint>
     <!-- Start: Port Surge -->
+    <link name="surge_port_servo_link"/>
+    <link name="surge_port_thruster_link"/>
     <link name="surge_port_duct_link"/>
-    <joint name="race2/surge_port_servo_joint" type="revolute">
+    <joint name="surge_port_servo_joint" type="fixed">
         <origin xyz="-0.86 -0.125 -0.05485" rpy="-1.5707 0.0 -0.52"/>
         <parent link="base_link"/>
+        <child link="surge_port_servo_link"/>
+    </joint>
+     <joint name="race2/surge_port_servo2duct_joint" type="revolute">
+        <origin xyz="0.0 0.0 0.0" rpy="0.0 0.0 0.0"/>
+        <parent link="surge_port_servo_link"/>
         <child link="surge_port_duct_link"/>
         <axis xyz="0 0 1"/>
         <limit effort="10" lower="-1.57" upper="1.57" velocity="10"/>
     </joint>
-    <!-- End: Port Surge -->
+    <joint name="surge_port_thruster_joint" type="fixed">
+        <origin rpy="0.0 0.0 0.0" xyz="0.0 0.0 0.0"/>
+        <parent link="surge_port_duct_link"/>
+        <child link="surge_port_thruster_link"/>
+    </joint>
     <!-- Start: Starboard Surge -->
-    <link name="surge_starbrd_duct_link"/>
+    <!-- <link name="surge_starboard_duct_link"/>
     <joint name="race2/surge_starboard_servo_joint" type="revolute">
         <origin xyz="-0.86 0.125 -0.05485" rpy="1.5707 0.0 0.52"/>
-        <parent link="base_link"/>
-        <child link="surge_starbrd_duct_link"/>
+        <parent link="cg_link"/>
+        <child link="surge_starboard_duct_link"/>
         <axis xyz="0 0 1"/>
         <limit effort="10" lower="-1.57" upper="1.57" velocity="10"/>
     </joint>
+    <link name="surge_starboard_base_link"/>
+    <joint name="surge_starboard_base_link" type="fixed">
+        <origin xyz="0.0 0.0 0.0" rpy="0 0.0 0.0"/>
+        <parent link="surge_starboard_duct_link"/>
+        <child link="surge_starboard_base_link"/>
+    </joint>
+    <link name="surge_starboard_thruster_link"/>
+    <joint name="race2/surge_starboard_thruster_joint" type="fixed">
+        <origin xyz="-0.86 0.125 -0.05485" rpy="1.5707 0.0 0.52"/>
+        <parent link="surge_port_base_link"/>
+        <child link="surge_starboard_thruster_link"/>
+    </joint> -->
     <!-- End: Starboard Surge -->
     <!-- Heave Bow Thruster -->
     <link name="heave_bow_thruster_link"/>
     <joint name="heave_bow_thruster_joint" type="fixed">
-        <origin xyz="-0.07535 0.0 -0.07535" rpy="0.0 1.57079632679 0.0"/>
+        <origin xyz="-0.07535 0.0 -0.07535" rpy="3.1415926 -1.571 0.0"/>
         <parent link="base_link"/>
         <child link="heave_bow_thruster_link"/>
@@ -81,5 +104,5 @@
     <link name="heave_stern_port_thruster_link"/>
     <joint name="heave_stern_port_thruster_joint" type="fixed">
-        <origin xyz="-0.56 -0.1034 -0.07535" rpy="0.0 1.57079632679 0.0"/>
+        <origin xyz="-0.56 -0.1034 -0.07535" rpy="-1.571 -1.571 0.0"/>
         <parent link="base_link"/>
         <child link="heave_stern_port_thruster_link"/>
@@ -88,5 +111,5 @@
     <link name="heave_stern_stbd_thruster_link"/>
     <joint name="heave_stern_stbd_thruster_joint" type="fixed">
-        <origin xyz="-0.56 0.1034 -0.07535" rpy="0.0 1.57079632679 0.0"/>
+        <origin xyz="-0.56 0.1034 -0.07535" rpy="1.571 -1.571 0.0"/>
         <parent link="base_link"/>
         <child link="heave_stern_stbd_thruster_link"/>
@@ -95,5 +118,5 @@
     <link name="sway_stern_thruster_link"/>
     <joint name="sway_stern_thruster_joint" type="fixed">
-        <origin xyz="-0.66635 0.0 -0.07535" rpy="0.0 0.0 -1.57079632679"/>
+        <origin xyz="-0.66635 0.0 -0.07535" rpy="3.1415926 0.0 -1.571"/>
         <parent link="base_link"/>
         <child link="sway_stern_thruster_link"/>

Commit message: startboard scn

File: race2_description/urdf/base.urdf.xacro (robot description, xacro)
@@ -1,3 +1,10 @@
 <?xml version="1.0"?>
+<!--
+    This file is part of RACE AUV project.
+    Author: Farhang Naderi, Mingxi Zhou
+    Email: farhang.nba@gmail.com,farhang.naderi@uri.edu,mzhou@uri.edu
+    Year: 2023
+    Copyright (C) 2023 Smart Ocean Systems Laboratory
+-->
 <robot name="race2" xmlns:xacro="http://ros.org/wiki/xacro">
     <link name="base_link">
@@ -73,4 +80,24 @@
     </joint>
     <!-- Start: Starboard Surge -->
+    <link name="surge_starboard_servo_link"/>
+    <link name="surge_starboard_thruster_link"/>
+    <link name="surge_starboard_duct_link"/>
+    <joint name="surge_starboard_servo_joint" type="fixed">
+        <origin xyz="-0.86 0.125 -0.05485" rpy="1.5707 0.0 0.52"/>
+        <parent link="base_link"/>
+        <child link="surge_starboard_servo_link"/>
+    </joint>
+     <joint name="race2/surge_starboard_servo2duct_joint" type="revolute">
+        <origin xyz="0.0 0.0 0.0" rpy="0.0 0.0 0.0"/>
+        <parent link="surge_starboard_servo_link"/>
+        <child link="surge_starboard_duct_link"/>
+        <axis xyz="0 0 1"/>
+        <limit effort="10" lower="-1.57" upper="1.57" velocity="10"/>
+    </joint>
+    <joint name="surge_starboard_thruster_joint" type="fixed">
+        <origin rpy="0.0 0.0 0.0" xyz="0.0 0.0 0.0"/>
+        <parent link="surge_starboard_duct_link"/>
+        <child link="surge_starboard_thruster_link"/>
+    </joint>
     <!-- <link name="surge_starboard_duct_link"/>
     <joint name="race2/surge_starboard_servo_joint" type="revolute">

Commit message: urdf and outdated files corrections

File: race2_description/urdf/base.urdf.xacro (robot description, xacro)
@@ -10,5 +10,5 @@
     <link name="base_link">
         <visual>
-            <origin xyz="0.0 0.0 0.0" rpy="0.0 0.0 0.0"/>
+            <origin xyz="0.0 0.0 0.0" rpy="3.1415926 0.0 0.0"/>
             <geometry>
                 <mesh filename="package://world_of_stonefish/data/parts/body/race2_body.obj" scale="1.0 1.0 1.0"/>
@@ -18,5 +18,5 @@
     <link name="cg_link"/>
     <joint name="cg_joint" type="fixed">
-        <origin xyz="0.0 0.0 0.0" rpy="3.1415926 0.0 0.0"/>
+        <origin xyz="-0.45 0.0 0.0" rpy="3.1415926 0.0 0.0"/>
         <parent link="base_link"/>
         <child link="cg_link"/>
@@ -24,5 +24,5 @@
     <link name="imu"/>
     <joint name="imu_joint" type="fixed">
-        <origin xyz="0.0 0.0 0.0" rpy="0.0 0.0 0.0"/>
+        <origin xyz="-0.49 0.0 0.05" rpy="3.1415926 0.0 0.0"/>
         <parent link="base_link"/>
         <child link="imu"/>
@@ -31,10 +31,10 @@
     <joint name="imu_sf_joint" type="fixed">
         <origin xyz="0.0 0.0 0.0" rpy="0.0 0.0 0.0"/>
-        <parent link="base_link"/>
+        <parent link="imu"/>
         <child link="imu_sf"/>
     </joint>
     <link name="dvl"/>
     <joint name="dvl_joint" type="fixed">
-        <origin xyz="-0.22 0.0 -0.08" rpy="3.1415926 0.0 0.0"/>
+        <origin xyz="-0.35 0.0 -0.08" rpy="3.1415926 0.0 0.0"/>
         <parent link="base_link"/>
         <child link="dvl"/>
@@ -42,5 +42,5 @@
     <link name="dvl_sf"/>
     <joint name="dvl_sf_joint" type="fixed">
-        <origin xyz="-0.22 0.0 -0.08" rpy="0.0 0.0 0.0"/>
+        <origin xyz="-0.35 0.0 -0.08" rpy="0.0 0.0 0.0"/>
         <parent link="base_link"/>
         <child link="dvl_sf"/>
@@ -58,4 +58,25 @@
         <child link="pressure"/>
     </joint>
+    <!-- Start: Starboard Surge -->
+    <link name="surge_starboard_servo_link"/>
+    <link name="surge_starboard_thruster_link"/>
+    <link name="surge_starboard_duct_link"/>
+    <joint name="surge_starboard_servo_joint" type="fixed">
+        <origin xyz="-0.79 -0.079 0.05485" rpy="1.5707 0.0 -0.52"/>
+        <parent link="base_link"/>
+        <child link="surge_starboard_servo_link"/>
+    </joint>
+     <joint name="race2/surge_starboard_servo2duct_joint" type="revolute">
+        <origin xyz="0.0 0.0 0.0" rpy="0.0 0.0 0.0"/>
+        <parent link="surge_starboard_servo_link"/>
+        <child link="surge_starboard_duct_link"/>
+        <axis xyz="0 0 1"/>
+        <limit effort="10" lower="-1.57" upper="1.57" velocity="10"/>
+    </joint>
+    <joint name="surge_starboard_thruster_joint" type="fixed">
+        <origin rpy="0.0 0.0 0.0" xyz="0.0 0.0 0.0"/>
+        <parent link="surge_starboard_duct_link"/>
+        <child link="surge_starboard_thruster_link"/>
+    </joint>
     <!-- Start: Port Surge -->
     <link name="surge_port_servo_link"/>
@@ -63,5 +84,5 @@
     <link name="surge_port_duct_link"/>
     <joint name="surge_port_servo_joint" type="fixed">
-        <origin xyz="-0.86 -0.125 -0.05485" rpy="-1.5707 0.0 -0.52"/>
+        <origin xyz="-0.79 0.079 0.05485" rpy="-1.5707 0.0 0.52"/>
         <parent link="base_link"/>
         <child link="surge_port_servo_link"/>
@@ -79,71 +100,30 @@
         <child link="surge_port_thruster_link"/>
     </joint>
-    <!-- Start: Starboard Surge -->
-    <link name="surge_starboard_servo_link"/>
-    <link name="surge_starboard_thruster_link"/>
-    <link name="surge_starboard_duct_link"/>
-    <joint name="surge_starboard_servo_joint" type="fixed">
-        <origin xyz="-0.86 0.125 -0.05485" rpy="1.5707 0.0 0.52"/>
-        <parent link="base_link"/>
-        <child link="surge_starboard_servo_link"/>
-    </joint>
-     <joint name="race2/surge_starboard_servo2duct_joint" type="revolute">
-        <origin xyz="0.0 0.0 0.0" rpy="0.0 0.0 0.0"/>
-        <parent link="surge_starboard_servo_link"/>
-        <child link="surge_starboard_duct_link"/>
-        <axis xyz="0 0 1"/>
-        <limit effort="10" lower="-1.57" upper="1.57" velocity="10"/>
-    </joint>
-    <joint name="surge_starboard_thruster_joint" type="fixed">
-        <origin rpy="0.0 0.0 0.0" xyz="0.0 0.0 0.0"/>
-        <parent link="surge_starboard_duct_link"/>
-        <child link="surge_starboard_thruster_link"/>
-    </joint>
-    <!-- <link name="surge_starboard_duct_link"/>
-    <joint name="race2/surge_starboard_servo_joint" type="revolute">
-        <origin xyz="-0.86 0.125 -0.05485" rpy="1.5707 0.0 0.52"/>
-        <parent link="cg_link"/>
-        <child link="surge_starboard_duct_link"/>
-        <axis xyz="0 0 1"/>
-        <limit effort="10" lower="-1.57" upper="1.57" velocity="10"/>
-    </joint>
-    <link name="surge_starboard_base_link"/>
-    <joint name="surge_starboard_base_link" type="fixed">
-        <origin xyz="0.0 0.0 0.0" rpy="0 0.0 0.0"/>
-        <parent link="surge_starboard_duct_link"/>
-        <child link="surge_starboard_base_link"/>
-    </joint>
-    <link name="surge_starboard_thruster_link"/>
-    <joint name="race2/surge_starboard_thruster_joint" type="fixed">
-        <origin xyz="-0.86 0.125 -0.05485" rpy="1.5707 0.0 0.52"/>
-        <parent link="surge_port_base_link"/>
-        <child link="surge_starboard_thruster_link"/>
-    </joint> -->
-    <!-- End: Starboard Surge -->
+    <!-- End: Port Surge -->
     <!-- Heave Bow Thruster -->
     <link name="heave_bow_thruster_link"/>
     <joint name="heave_bow_thruster_joint" type="fixed">
-        <origin xyz="-0.07535 0.0 -0.07535" rpy="3.1415926 -1.571 0.0"/>
+        <origin xyz="-0.076 0.0 0.086" rpy="-1.571 1.571 0.0"/>
         <parent link="base_link"/>
         <child link="heave_bow_thruster_link"/>
     </joint>
     <!-- Heave Stern Thruster Port -->
-    <link name="heave_stern_port_thruster_link"/>
+    <!-- <link name="heave_stern_port_thruster_link"/>
     <joint name="heave_stern_port_thruster_joint" type="fixed">
         <origin xyz="-0.56 -0.1034 -0.07535" rpy="-1.571 -1.571 0.0"/>
         <parent link="base_link"/>
         <child link="heave_stern_port_thruster_link"/>
-    </joint>
+    </joint> -->
     <!-- Heave Stern Thruster Stbd -->
-    <link name="heave_stern_stbd_thruster_link"/>
+    <!-- <link name="heave_stern_stbd_thruster_link"/>
     <joint name="heave_stern_stbd_thruster_joint" type="fixed">
         <origin xyz="-0.56 0.1034 -0.07535" rpy="1.571 -1.571 0.0"/>
         <parent link="base_link"/>
         <child link="heave_stern_stbd_thruster_link"/>
-    </joint>
+    </joint> -->
     <!-- Sway Stern Thruster -->
     <link name="sway_stern_thruster_link"/>
     <joint name="sway_stern_thruster_joint" type="fixed">
-        <origin xyz="-0.66635 0.0 -0.07535" rpy="3.1415926 0.0 -1.571"/>
+        <origin xyz="-0.66635 0.0 0.07535" rpy="3.1415926 0.0 -1.571"/>
         <parent link="base_link"/>
         <child link="sway_stern_thruster_link"/>

Commit message: debugging. problem found was mainly the PID controller

File: race2_description/urdf/base.urdf.xacro (robot description, xacro)
@@ -10,5 +10,5 @@
     <link name="base_link">
         <visual>
-            <origin xyz="0.0 0.0 0.0" rpy="3.1415926 0.0 0.0"/>
+            <origin xyz="0.45 0.0 0.0" rpy="3.1415926 0.0 0.0"/>
             <geometry>
                 <mesh filename="package://world_of_stonefish/data/parts/body/race2_body.obj" scale="1.0 1.0 1.0"/>
@@ -18,5 +18,5 @@
     <link name="cg_link"/>
     <joint name="cg_joint" type="fixed">
-        <origin xyz="-0.45 0.0 0.0" rpy="3.1415926 0.0 0.0"/>
+        <origin xyz="-0.0 0.0 0.0" rpy="3.1415926 0.0 0.0"/>
         <parent link="base_link"/>
         <child link="cg_link"/>
@@ -24,5 +24,5 @@
     <link name="imu"/>
     <joint name="imu_joint" type="fixed">
-        <origin xyz="-0.49 0.0 0.05" rpy="3.1415926 0.0 0.0"/>
+        <origin xyz="-0.04 0.0 0.05" rpy="3.1415926 0.0 0.0"/>
         <parent link="base_link"/>
         <child link="imu"/>
@@ -36,5 +36,5 @@
     <link name="dvl"/>
     <joint name="dvl_joint" type="fixed">
-        <origin xyz="-0.35 0.0 -0.08" rpy="3.1415926 0.0 0.0"/>
+        <origin xyz="0.1 0.0 0.0" rpy="3.1415926 0.0 0.0"/>
         <parent link="base_link"/>
         <child link="dvl"/>
@@ -42,5 +42,5 @@
     <link name="dvl_sf"/>
     <joint name="dvl_sf_joint" type="fixed">
-        <origin xyz="-0.35 0.0 -0.08" rpy="0.0 0.0 0.0"/>
+        <origin xyz="0.1 0.0 0.0" rpy="0.0 0.0 0.0"/>
         <parent link="base_link"/>
         <child link="dvl_sf"/>
@@ -54,5 +54,5 @@
     <link name="pressure"/>
     <joint name="pressure_joint" type="fixed">
-        <origin xyz="-0.25 0.0 0.05" rpy="3.1415926 0.0 0.0"/>
+        <origin xyz="0.2 0.0 0.05" rpy="3.1415926 0.0 0.0"/>
         <parent link="base_link"/>
         <child link="pressure"/>
@@ -63,5 +63,5 @@
     <link name="surge_starboard_duct_link"/>
     <joint name="surge_starboard_servo_joint" type="fixed">
-        <origin xyz="-0.79 -0.079 0.05485" rpy="1.5707 0.0 -0.52"/>
+        <origin xyz="-0.34 -0.079 0.05485" rpy="1.5707 0.0 -0.52"/>
         <parent link="base_link"/>
         <child link="surge_starboard_servo_link"/>
@@ -84,5 +84,5 @@
     <link name="surge_port_duct_link"/>
     <joint name="surge_port_servo_joint" type="fixed">
-        <origin xyz="-0.79 0.079 0.05485" rpy="-1.5707 0.0 0.52"/>
+        <origin xyz="-0.34 0.079 0.05485" rpy="-1.5707 0.0 0.52"/>
         <parent link="base_link"/>
         <child link="surge_port_servo_link"/>
@@ -104,5 +104,5 @@
     <link name="heave_bow_thruster_link"/>
     <joint name="heave_bow_thruster_joint" type="fixed">
-        <origin xyz="-0.076 0.0 0.086" rpy="-1.571 1.571 0.0"/>
+        <origin xyz="0.374 0.0 0.086" rpy="-1.571 1.571 0.0"/>
         <parent link="base_link"/>
         <child link="heave_bow_thruster_link"/>
@@ -125,5 +125,5 @@
     <link name="sway_stern_thruster_link"/>
     <joint name="sway_stern_thruster_joint" type="fixed">
-        <origin xyz="-0.66635 0.0 0.07535" rpy="3.1415926 0.0 -1.571"/>
+        <origin xyz="-0.216 0.0 0.07535" rpy="3.1415926 0.0 -1.571"/>
         <parent link="base_link"/>
         <child link="sway_stern_thruster_link"/>

Commit message: adjusted urdf to move the surge thruster links outward

File: race2_description/urdf/base.urdf.xacro (robot description, xacro)
@@ -68,5 +68,5 @@
     </joint>
      <joint name="race2/surge_starboard_servo2duct_joint" type="revolute">
-        <origin xyz="0.0 0.0 0.0" rpy="0.0 0.0 0.0"/>
+        <origin xyz="0.0 0.0 0.07" rpy="0.0 0.0 0.0"/>
         <parent link="surge_starboard_servo_link"/>
         <child link="surge_starboard_duct_link"/>
@@ -89,5 +89,5 @@
     </joint>
      <joint name="race2/surge_port_servo2duct_joint" type="revolute">
-        <origin xyz="0.0 0.0 0.0" rpy="0.0 0.0 0.0"/>
+        <origin xyz="0.0 0.0 0.07" rpy="0.0 0.0 0.0"/>
         <parent link="surge_port_servo_link"/>
         <child link="surge_port_duct_link"/>
