Commit message: Control and URDF update!

File: race2_description/urdf/base.urdf.xacro (robot description, xacro)
@@ -10,101 +10,102 @@
     <link name="base_link">
         <visual>
-            <origin xyz="0.45 0.0 0.0" rpy="3.1415926 0.0 0.0"/>
+            <origin xyz="0.45 0.0 0.0" rpy="3.1415926 0.0 0.0" />
             <geometry>
-                <mesh filename="package://world_of_stonefish/data/parts/body/race2_body.obj" scale="1.0 1.0 1.0"/>
+                <mesh filename="package://world_of_stonefish/data/parts/body/race2_body.obj"
+                    scale="1.0 1.0 1.0" />
             </geometry>
         </visual>
     </link>
-    <link name="cg_link"/>
+    <link name="cg_link" />
     <joint name="cg_joint" type="fixed">
-        <origin xyz="-0.0 0.0 0.0" rpy="3.1415926 0.0 0.0"/>
-        <parent link="base_link"/>
-        <child link="cg_link"/>
+        <origin xyz="-0.0 0.0 0.0" rpy="3.1415926 0.0 0.0" />
+        <parent link="base_link" />
+        <child link="cg_link" />
     </joint>
-    <link name="imu"/>
+    <link name="imu" />
     <joint name="imu_joint" type="fixed">
-        <origin xyz="-0.04 0.0 0.05" rpy="3.1415926 0.0 0.0"/>
-        <parent link="base_link"/>
-        <child link="imu"/>
+        <origin xyz="-0.04 0.0 0.05" rpy="3.1415926 0.0 0.0" />
+        <parent link="base_link" />
+        <child link="imu" />
     </joint>
-    <link name="imu_sf"/>
+    <link name="imu_sf" />
     <joint name="imu_sf_joint" type="fixed">
-        <origin xyz="0.0 0.0 0.0" rpy="0.0 0.0 0.0"/>
-        <parent link="imu"/>
-        <child link="imu_sf"/>
+        <origin xyz="0.0 0.0 0.0" rpy="0.0 0.0 0.0" />
+        <parent link="imu" />
+        <child link="imu_sf" />
     </joint>
-    <link name="dvl"/>
+    <link name="dvl" />
     <joint name="dvl_joint" type="fixed">
-        <origin xyz="0.1 0.0 0.0" rpy="3.1415926 0.0 0.0"/>
-        <parent link="base_link"/>
-        <child link="dvl"/>
+        <origin xyz="0.1 0.0 0.0" rpy="3.1415926 0.0 0.0" />
+        <parent link="base_link" />
+        <child link="dvl" />
     </joint>
-    <link name="dvl_sf"/>
+    <link name="dvl_sf" />
     <joint name="dvl_sf_joint" type="fixed">
-        <origin xyz="0.1 0.0 0.0" rpy="0.0 0.0 0.0"/>
-        <parent link="base_link"/>
-        <child link="dvl_sf"/>
+        <origin xyz="0.1 0.0 0.0" rpy="0.0 0.0 0.0" />
+        <parent link="base_link" />
+        <child link="dvl_sf" />
     </joint>
-    <link name="gps"/>
+    <link name="gps" />
     <joint name="gps_joint" type="fixed">
-        <origin xyz="0.0 0.0 0.28" rpy="3.14 0.0 -1.5707963"/>
-        <parent link="base_link"/>
-        <child link="gps"/>
+        <origin xyz="0.0 0.0 0.28" rpy="3.14 0.0 -1.5707963" />
+        <parent link="base_link" />
+        <child link="gps" />
     </joint>
-    <link name="pressure"/>
+    <link name="pressure" />
     <joint name="pressure_joint" type="fixed">
-        <origin xyz="0.2 0.0 0.05" rpy="3.1415926 0.0 0.0"/>
-        <parent link="base_link"/>
-        <child link="pressure"/>
+        <origin xyz="0.2 0.0 0.05" rpy="3.1415926 0.0 0.0" />
+        <parent link="base_link" />
+        <child link="pressure" />
     </joint>
+    <!-- Start: Port Surge -->
+    <link name="surge_port_servo_link" />
+    <link name="surge_port_thruster_link" />
+    <link name="surge_port_duct_link" />
+    <joint name="surge_port_servo_joint" type="fixed">
+        <origin xyz="-0.34 0.079 0.05485" rpy="-1.5707 0.0 0.52" />
+        <parent link="base_link" />
+        <child link="surge_port_servo_link" />
+    </joint>
+    <joint name="race2/surge_port_servo2duct_joint" type="revolute">
+        <origin xyz="0.0 0.0 0.07" rpy="0.0 0.0 0.0" />
+        <parent link="surge_port_servo_link" />
+        <child link="surge_port_duct_link" />
+        <axis xyz="0 0 1" />
+        <limit effort="10" lower="-1.57" upper="1.57" velocity="10" />
+    </joint>
+    <joint name="surge_port_thruster_joint" type="fixed">
+        <origin rpy="0.0 0.0 0.0" xyz="0.0 0.0 0.0" />
+        <parent link="surge_port_duct_link" />
+        <child link="surge_port_thruster_link" />
+    </joint>
+    <!-- End: Port Surge -->
     <!-- Start: Starboard Surge -->
-    <link name="surge_starboard_servo_link"/>
-    <link name="surge_starboard_thruster_link"/>
-    <link name="surge_starboard_duct_link"/>
+    <link name="surge_starboard_servo_link" />
+    <link name="surge_starboard_thruster_link" />
+    <link name="surge_starboard_duct_link" />
     <joint name="surge_starboard_servo_joint" type="fixed">
-        <origin xyz="-0.34 -0.079 0.05485" rpy="1.5707 0.0 -0.52"/>
-        <parent link="base_link"/>
-        <child link="surge_starboard_servo_link"/>
+        <origin xyz="-0.34 -0.079 0.05485" rpy="1.5707 0.0 -0.52" />
+        <parent link="base_link" />
+        <child link="surge_starboard_servo_link" />
     </joint>
-     <joint name="race2/surge_starboard_servo2duct_joint" type="revolute">
-        <origin xyz="0.0 0.0 0.07" rpy="0.0 0.0 0.0"/>
-        <parent link="surge_starboard_servo_link"/>
-        <child link="surge_starboard_duct_link"/>
-        <axis xyz="0 0 1"/>
-        <limit effort="10" lower="-1.57" upper="1.57" velocity="10"/>
+    <joint name="race2/surge_starboard_servo2duct_joint" type="revolute">
+        <origin xyz="0.0 0.0 0.07" rpy="0.0 0.0 0.0" />
+        <parent link="surge_starboard_servo_link" />
+        <child link="surge_starboard_duct_link" />
+        <axis xyz="0 0 1" />
+        <limit effort="10" lower="-1.57" upper="1.57" velocity="10" />
     </joint>
     <joint name="surge_starboard_thruster_joint" type="fixed">
-        <origin rpy="0.0 0.0 0.0" xyz="0.0 0.0 0.0"/>
-        <parent link="surge_starboard_duct_link"/>
-        <child link="surge_starboard_thruster_link"/>
+        <origin rpy="0.0 0.0 0.0" xyz="0.0 0.0 0.0" />
+        <parent link="surge_starboard_duct_link" />
+        <child link="surge_starboard_thruster_link" />
     </joint>
-    <!-- Start: Port Surge -->
-    <link name="surge_port_servo_link"/>
-    <link name="surge_port_thruster_link"/>
-    <link name="surge_port_duct_link"/>
-    <joint name="surge_port_servo_joint" type="fixed">
-        <origin xyz="-0.34 0.079 0.05485" rpy="-1.5707 0.0 0.52"/>
-        <parent link="base_link"/>
-        <child link="surge_port_servo_link"/>
-    </joint>
-     <joint name="race2/surge_port_servo2duct_joint" type="revolute">
-        <origin xyz="0.0 0.0 0.07" rpy="0.0 0.0 0.0"/>
-        <parent link="surge_port_servo_link"/>
-        <child link="surge_port_duct_link"/>
-        <axis xyz="0 0 1"/>
-        <limit effort="10" lower="-1.57" upper="1.57" velocity="10"/>
-    </joint>
-    <joint name="surge_port_thruster_joint" type="fixed">
-        <origin rpy="0.0 0.0 0.0" xyz="0.0 0.0 0.0"/>
-        <parent link="surge_port_duct_link"/>
-        <child link="surge_port_thruster_link"/>
-    </joint>
-    <!-- End: Port Surge -->
     <!-- Heave Bow Thruster -->
-    <link name="heave_bow_thruster_link"/>
+    <link name="heave_bow_thruster_link" />
     <joint name="heave_bow_thruster_joint" type="fixed">
-        <origin xyz="0.374 0.0 0.086" rpy="-1.571 1.571 0.0"/>
-        <parent link="base_link"/>
-        <child link="heave_bow_thruster_link"/>
+        <origin xyz="0.374 0.0 0.086" rpy="3.1415926 1.571 0.0" />
+        <parent link="base_link" />
+        <child link="heave_bow_thruster_link" />
     </joint>
     <!-- Heave Stern Thruster Port -->
@@ -123,9 +124,9 @@
     </joint> -->
     <!-- Sway Stern Thruster -->
-    <link name="sway_stern_thruster_link"/>
+    <link name="sway_stern_thruster_link" />
     <joint name="sway_stern_thruster_joint" type="fixed">
-        <origin xyz="-0.216 0.0 0.07535" rpy="3.1415926 0.0 -1.571"/>
-        <parent link="base_link"/>
-        <child link="sway_stern_thruster_link"/>
+        <origin xyz="-0.216 0.0 0.07535" rpy="3.1415926 0.0 -1.571" />
+        <parent link="base_link" />
+        <child link="sway_stern_thruster_link" />
     </joint>
     <!-- perception sensors -->

Commit message: Revert "Control and URDF update!"
This reverts commit 30fec4451f6d0baae57f831ab167ea010f445c8b.

File: race2_description/urdf/base.urdf.xacro (robot description, xacro)
@@ -10,102 +10,101 @@
     <link name="base_link">
         <visual>
-            <origin xyz="0.45 0.0 0.0" rpy="3.1415926 0.0 0.0" />
+            <origin xyz="0.45 0.0 0.0" rpy="3.1415926 0.0 0.0"/>
             <geometry>
-                <mesh filename="package://world_of_stonefish/data/parts/body/race2_body.obj"
-                    scale="1.0 1.0 1.0" />
+                <mesh filename="package://world_of_stonefish/data/parts/body/race2_body.obj" scale="1.0 1.0 1.0"/>
             </geometry>
         </visual>
     </link>
-    <link name="cg_link" />
+    <link name="cg_link"/>
     <joint name="cg_joint" type="fixed">
-        <origin xyz="-0.0 0.0 0.0" rpy="3.1415926 0.0 0.0" />
-        <parent link="base_link" />
-        <child link="cg_link" />
+        <origin xyz="-0.0 0.0 0.0" rpy="3.1415926 0.0 0.0"/>
+        <parent link="base_link"/>
+        <child link="cg_link"/>
     </joint>
-    <link name="imu" />
+    <link name="imu"/>
     <joint name="imu_joint" type="fixed">
-        <origin xyz="-0.04 0.0 0.05" rpy="3.1415926 0.0 0.0" />
-        <parent link="base_link" />
-        <child link="imu" />
+        <origin xyz="-0.04 0.0 0.05" rpy="3.1415926 0.0 0.0"/>
+        <parent link="base_link"/>
+        <child link="imu"/>
     </joint>
-    <link name="imu_sf" />
+    <link name="imu_sf"/>
     <joint name="imu_sf_joint" type="fixed">
-        <origin xyz="0.0 0.0 0.0" rpy="0.0 0.0 0.0" />
-        <parent link="imu" />
-        <child link="imu_sf" />
+        <origin xyz="0.0 0.0 0.0" rpy="0.0 0.0 0.0"/>
+        <parent link="imu"/>
+        <child link="imu_sf"/>
     </joint>
-    <link name="dvl" />
+    <link name="dvl"/>
     <joint name="dvl_joint" type="fixed">
-        <origin xyz="0.1 0.0 0.0" rpy="3.1415926 0.0 0.0" />
-        <parent link="base_link" />
-        <child link="dvl" />
+        <origin xyz="0.1 0.0 0.0" rpy="3.1415926 0.0 0.0"/>
+        <parent link="base_link"/>
+        <child link="dvl"/>
     </joint>
-    <link name="dvl_sf" />
+    <link name="dvl_sf"/>
     <joint name="dvl_sf_joint" type="fixed">
-        <origin xyz="0.1 0.0 0.0" rpy="0.0 0.0 0.0" />
-        <parent link="base_link" />
-        <child link="dvl_sf" />
+        <origin xyz="0.1 0.0 0.0" rpy="0.0 0.0 0.0"/>
+        <parent link="base_link"/>
+        <child link="dvl_sf"/>
     </joint>
-    <link name="gps" />
+    <link name="gps"/>
     <joint name="gps_joint" type="fixed">
-        <origin xyz="0.0 0.0 0.28" rpy="3.14 0.0 -1.5707963" />
-        <parent link="base_link" />
-        <child link="gps" />
+        <origin xyz="0.0 0.0 0.28" rpy="3.14 0.0 -1.5707963"/>
+        <parent link="base_link"/>
+        <child link="gps"/>
     </joint>
-    <link name="pressure" />
+    <link name="pressure"/>
     <joint name="pressure_joint" type="fixed">
-        <origin xyz="0.2 0.0 0.05" rpy="3.1415926 0.0 0.0" />
-        <parent link="base_link" />
-        <child link="pressure" />
+        <origin xyz="0.2 0.0 0.05" rpy="3.1415926 0.0 0.0"/>
+        <parent link="base_link"/>
+        <child link="pressure"/>
+    </joint>
+    <!-- Start: Starboard Surge -->
+    <link name="surge_starboard_servo_link"/>
+    <link name="surge_starboard_thruster_link"/>
+    <link name="surge_starboard_duct_link"/>
+    <joint name="surge_starboard_servo_joint" type="fixed">
+        <origin xyz="-0.34 -0.079 0.05485" rpy="1.5707 0.0 -0.52"/>
+        <parent link="base_link"/>
+        <child link="surge_starboard_servo_link"/>
+    </joint>
+     <joint name="race2/surge_starboard_servo2duct_joint" type="revolute">
+        <origin xyz="0.0 0.0 0.07" rpy="0.0 0.0 0.0"/>
+        <parent link="surge_starboard_servo_link"/>
+        <child link="surge_starboard_duct_link"/>
+        <axis xyz="0 0 1"/>
+        <limit effort="10" lower="-1.57" upper="1.57" velocity="10"/>
+    </joint>
+    <joint name="surge_starboard_thruster_joint" type="fixed">
+        <origin rpy="0.0 0.0 0.0" xyz="0.0 0.0 0.0"/>
+        <parent link="surge_starboard_duct_link"/>
+        <child link="surge_starboard_thruster_link"/>
     </joint>
     <!-- Start: Port Surge -->
-    <link name="surge_port_servo_link" />
-    <link name="surge_port_thruster_link" />
-    <link name="surge_port_duct_link" />
+    <link name="surge_port_servo_link"/>
+    <link name="surge_port_thruster_link"/>
+    <link name="surge_port_duct_link"/>
     <joint name="surge_port_servo_joint" type="fixed">
-        <origin xyz="-0.34 0.079 0.05485" rpy="-1.5707 0.0 0.52" />
-        <parent link="base_link" />
-        <child link="surge_port_servo_link" />
+        <origin xyz="-0.34 0.079 0.05485" rpy="-1.5707 0.0 0.52"/>
+        <parent link="base_link"/>
+        <child link="surge_port_servo_link"/>
     </joint>
-    <joint name="race2/surge_port_servo2duct_joint" type="revolute">
-        <origin xyz="0.0 0.0 0.07" rpy="0.0 0.0 0.0" />
-        <parent link="surge_port_servo_link" />
-        <child link="surge_port_duct_link" />
-        <axis xyz="0 0 1" />
-        <limit effort="10" lower="-1.57" upper="1.57" velocity="10" />
+     <joint name="race2/surge_port_servo2duct_joint" type="revolute">
+        <origin xyz="0.0 0.0 0.07" rpy="0.0 0.0 0.0"/>
+        <parent link="surge_port_servo_link"/>
+        <child link="surge_port_duct_link"/>
+        <axis xyz="0 0 1"/>
+        <limit effort="10" lower="-1.57" upper="1.57" velocity="10"/>
     </joint>
     <joint name="surge_port_thruster_joint" type="fixed">
-        <origin rpy="0.0 0.0 0.0" xyz="0.0 0.0 0.0" />
-        <parent link="surge_port_duct_link" />
-        <child link="surge_port_thruster_link" />
+        <origin rpy="0.0 0.0 0.0" xyz="0.0 0.0 0.0"/>
+        <parent link="surge_port_duct_link"/>
+        <child link="surge_port_thruster_link"/>
     </joint>
     <!-- End: Port Surge -->
-    <!-- Start: Starboard Surge -->
-    <link name="surge_starboard_servo_link" />
-    <link name="surge_starboard_thruster_link" />
-    <link name="surge_starboard_duct_link" />
-    <joint name="surge_starboard_servo_joint" type="fixed">
-        <origin xyz="-0.34 -0.079 0.05485" rpy="1.5707 0.0 -0.52" />
-        <parent link="base_link" />
-        <child link="surge_starboard_servo_link" />
-    </joint>
-    <joint name="race2/surge_starboard_servo2duct_joint" type="revolute">
-        <origin xyz="0.0 0.0 0.07" rpy="0.0 0.0 0.0" />
-        <parent link="surge_starboard_servo_link" />
-        <child link="surge_starboard_duct_link" />
-        <axis xyz="0 0 1" />
-        <limit effort="10" lower="-1.57" upper="1.57" velocity="10" />
-    </joint>
-    <joint name="surge_starboard_thruster_joint" type="fixed">
-        <origin rpy="0.0 0.0 0.0" xyz="0.0 0.0 0.0" />
-        <parent link="surge_starboard_duct_link" />
-        <child link="surge_starboard_thruster_link" />
-    </joint>
     <!-- Heave Bow Thruster -->
-    <link name="heave_bow_thruster_link" />
+    <link name="heave_bow_thruster_link"/>
     <joint name="heave_bow_thruster_joint" type="fixed">
-        <origin xyz="0.374 0.0 0.086" rpy="3.1415926 1.571 0.0" />
-        <parent link="base_link" />
-        <child link="heave_bow_thruster_link" />
+        <origin xyz="0.374 0.0 0.086" rpy="-1.571 1.571 0.0"/>
+        <parent link="base_link"/>
+        <child link="heave_bow_thruster_link"/>
     </joint>
     <!-- Heave Stern Thruster Port -->
@@ -124,9 +123,9 @@
     </joint> -->
     <!-- Sway Stern Thruster -->
-    <link name="sway_stern_thruster_link" />
+    <link name="sway_stern_thruster_link"/>
     <joint name="sway_stern_thruster_joint" type="fixed">
-        <origin xyz="-0.216 0.0 0.07535" rpy="3.1415926 0.0 -1.571" />
-        <parent link="base_link" />
-        <child link="sway_stern_thruster_link" />
+        <origin xyz="-0.216 0.0 0.07535" rpy="3.1415926 0.0 -1.571"/>
+        <parent link="base_link"/>
+        <child link="sway_stern_thruster_link"/>
     </joint>
     <!-- perception sensors -->

Commit message: Linear coeffs revert PR Draft!

File: race2_description/urdf/base.urdf.xacro (robot description, xacro)
@@ -76,5 +76,5 @@
     </joint>
     <joint name="surge_port_thruster_joint" type="fixed">
-        <origin rpy="0.0 0.0 0.0" xyz="0.0 0.0 0.0" />
+        <origin rpy="0.0 0.0 -1.78" xyz="0.0 0.0 0.0" />
         <parent link="surge_port_duct_link" />
         <child link="surge_port_thruster_link" />
@@ -98,5 +98,5 @@
     </joint>
     <joint name="surge_starboard_thruster_joint" type="fixed">
-        <origin rpy="0.0 0.0 0.0" xyz="0.0 0.0 0.0" />
+        <origin rpy="0.0 0.0 -1.78" xyz="0.0 0.0 0.0" />
         <parent link="surge_starboard_duct_link" />
         <child link="surge_starboard_thruster_link" />

Commit message: Angles slope correction based on hardware

File: race2_description/urdf/base.urdf.xacro (robot description, xacro)
@@ -64,5 +64,5 @@
     <link name="surge_port_duct_link" />
     <joint name="surge_port_servo_joint" type="fixed">
-        <origin xyz="-0.34 0.079 0.05485" rpy="-1.5707 0.0 0.52" />
+        <origin xyz="-0.34 0.079 0.05485" rpy="-1.5707 -1.78 0.52" />
         <parent link="base_link" />
         <child link="surge_port_servo_link" />
@@ -76,5 +76,5 @@
     </joint>
     <joint name="surge_port_thruster_joint" type="fixed">
-        <origin rpy="0.0 0.0 -1.78" xyz="0.0 0.0 0.0" />
+        <origin rpy="0.0 0.0 0.0" xyz="0.0 0.0 0.0" />
         <parent link="surge_port_duct_link" />
         <child link="surge_port_thruster_link" />
@@ -86,5 +86,5 @@
     <link name="surge_starboard_duct_link" />
     <joint name="surge_starboard_servo_joint" type="fixed">
-        <origin xyz="-0.34 -0.079 0.05485" rpy="1.5707 0.0 -0.52" />
+        <origin xyz="-0.34 -0.079 0.05485" rpy="1.5707 1.78 -0.52" />
         <parent link="base_link" />
         <child link="surge_starboard_servo_link" />
@@ -98,5 +98,5 @@
     </joint>
     <joint name="surge_starboard_thruster_joint" type="fixed">
-        <origin rpy="0.0 0.0 -1.78" xyz="0.0 0.0 0.0" />
+        <origin rpy="0.0 0.0 0.0" xyz="0.0 0.0 0.0" />
         <parent link="surge_starboard_duct_link" />
         <child link="surge_starboard_thruster_link" />

Commit message: - Changes to catch up with latest mvp control updates - More files for the vehicle launch

File: race2_description/urdf/base.urdf.xacro (robot description, xacro)
@@ -73,5 +73,5 @@
         <child link="surge_port_duct_link" />
         <axis xyz="0 0 1" />
-        <limit effort="10" lower="-3.14" upper="3.14" velocity="10" />
+        <limit effort="10" lower="-3.0" upper="3.0" velocity="10" />
     </joint>
     <joint name="surge_port_thruster_joint" type="fixed">
@@ -95,5 +95,5 @@
         <child link="surge_starboard_duct_link" />
         <axis xyz="0 0 1" />
-        <limit effort="10" lower="-3.14" upper="3.14" velocity="10" />
+        <limit effort="10" lower="-3.0" upper="3.0" velocity="10" />
     </joint>
     <joint name="surge_starboard_thruster_joint" type="fixed">

Commit message: editing control stuff rev1

File: race2_description/urdf/base.urdf.xacro (robot description, xacro)
@@ -73,5 +73,5 @@
         <child link="surge_port_duct_link" />
         <axis xyz="0 0 1" />
-        <limit effort="10" lower="-3.0" upper="3.0" velocity="10" />
+        <limit effort="10" lower="-2.1" upper="2.1" velocity="20" />
     </joint>
     <joint name="surge_port_thruster_joint" type="fixed">
@@ -95,5 +95,5 @@
         <child link="surge_starboard_duct_link" />
         <axis xyz="0 0 1" />
-        <limit effort="10" lower="-3.0" upper="3.0" velocity="10" />
+        <limit effort="10" lower="-2.1" upper="2.1" velocity="20" />
     </joint>
     <joint name="surge_starboard_thruster_joint" type="fixed">

Commit message: tuning

File: race2_description/urdf/base.urdf.xacro (robot description, xacro)
@@ -43,5 +43,5 @@
     <link name="dvl_sf" />
     <joint name="dvl_sf_joint" type="fixed">
-        <origin xyz="0.1 0.0 0.0" rpy="0.0 0.0 0.0" />
+        <origin xyz="0.0 0.0 0.0" rpy="0.0 0.0 0.0" />
         <parent link="base_link" />
         <child link="dvl_sf" />
@@ -73,5 +73,5 @@
         <child link="surge_port_duct_link" />
         <axis xyz="0 0 1" />
-        <limit effort="10" lower="-2.1" upper="2.1" velocity="20" />
+        <limit effort="10" lower="-2.0" upper="2.0" velocity="20" />
     </joint>
     <joint name="surge_port_thruster_joint" type="fixed">
@@ -95,5 +95,5 @@
         <child link="surge_starboard_duct_link" />
         <axis xyz="0 0 1" />
-        <limit effort="10" lower="-2.1" upper="2.1" velocity="20" />
+        <limit effort="10" lower="-2.0" upper="2.0" velocity="20" />
     </joint>
     <joint name="surge_starboard_thruster_joint" type="fixed">

Commit message: - integral windup config file for sim update - dvl SF position change - no joy temp timeout change

File: race2_description/urdf/base.urdf.xacro (robot description, xacro)
@@ -43,5 +43,5 @@
     <link name="dvl_sf" />
     <joint name="dvl_sf_joint" type="fixed">
-        <origin xyz="0.0 0.0 0.0" rpy="0.0 0.0 0.0" />
+        <origin xyz="0.1 0.0 0.0" rpy="0.0 0.0 0.0" />
         <parent link="base_link" />
         <child link="dvl_sf" />
@@ -73,5 +73,5 @@
         <child link="surge_port_duct_link" />
         <axis xyz="0 0 1" />
-        <limit effort="10" lower="-2.0" upper="2.0" velocity="20" />
+        <limit effort="10" lower="-3.0" upper="3.0" velocity="20" />
     </joint>
     <joint name="surge_port_thruster_joint" type="fixed">
@@ -95,5 +95,5 @@
         <child link="surge_starboard_duct_link" />
         <axis xyz="0 0 1" />
-        <limit effort="10" lower="-2.0" upper="2.0" velocity="20" />
+        <limit effort="10" lower="-3.0" upper="3.0" velocity="20" />
     </joint>
     <joint name="surge_starboard_thruster_joint" type="fixed">

Commit message: PID tuning for 5Hz controller

File: race2_description/urdf/base.urdf.xacro (robot description, xacro)
@@ -73,5 +73,5 @@
         <child link="surge_port_duct_link" />
         <axis xyz="0 0 1" />
-        <limit effort="10" lower="-3.0" upper="3.0" velocity="20" />
+        <limit effort="10" lower="-3.12" upper="3.12" velocity="20" />
     </joint>
     <joint name="surge_port_thruster_joint" type="fixed">
@@ -95,5 +95,5 @@
         <child link="surge_starboard_duct_link" />
         <axis xyz="0 0 1" />
-        <limit effort="10" lower="-3.0" upper="3.0" velocity="20" />
+        <limit effort="10" lower="-3.12" upper="3.12" velocity="20" />
     </joint>
     <joint name="surge_starboard_thruster_joint" type="fixed">
