Commit message: new pid values

File: race2_description/urdf/base.urdf.xacro (robot description, xacro)
@@ -64,5 +64,6 @@
     <link name="surge_port_duct_link" />
     <joint name="surge_port_servo_joint" type="fixed">
-        <origin xyz="-0.34 0.079 0.05485" rpy="-1.5707 -1.78 0.52" />
+        <!-- <origin xyz="-0.34 0.079 0.05485" rpy="-1.5707 -1.78 0.52" /> -->
+         <origin xyz="-0.34 0.079 0.05485" rpy="-1.5707 -0.21 0.52" />
         <parent link="base_link" />
         <child link="surge_port_servo_link" />
@@ -73,5 +74,5 @@
         <child link="surge_port_duct_link" />
         <axis xyz="0 0 1" />
-        <limit effort="10" lower="-3.12" upper="3.12" velocity="20" />
+        <limit effort="10" lower="-3.10000000000000" upper="3.10000000000000" velocity="20" />
     </joint>
     <joint name="surge_port_thruster_joint" type="fixed">
@@ -86,5 +87,6 @@
     <link name="surge_starboard_duct_link" />
     <joint name="surge_starboard_servo_joint" type="fixed">
-        <origin xyz="-0.34 -0.079 0.05485" rpy="1.5707 1.78 -0.52" />
+        <!-- <origin xyz="-0.34 -0.079 0.05485" rpy="1.5707 1.78 -0.52" /> -->
+         <origin xyz="-0.34 -0.079 0.05485" rpy="1.5707 0.21 -0.52" />
         <parent link="base_link" />
         <child link="surge_starboard_servo_link" />
@@ -95,5 +97,5 @@
         <child link="surge_starboard_duct_link" />
         <axis xyz="0 0 1" />
-        <limit effort="10" lower="-3.12" upper="3.12" velocity="20" />
+        <limit effort="10" lower="-3.10000000000000" upper="3.10000000000000" velocity="20" />
     </joint>
     <joint name="surge_starboard_thruster_joint" type="fixed">
@@ -149,5 +151,6 @@
     <link name="sway_stern_thruster_link" />
     <joint name="sway_stern_thruster_joint" type="fixed">
-        <origin xyz="-0.216 0.0 0.07535" rpy="3.1415926 0.0 -1.571" />
+        <origin xyz="-0.216 0.0 -0.07535" rpy="3.1415926 0.0 -1.571" />
+        <!-- <origin xyz="-0.216 0.0 0.0" rpy="3.1415926 0.0 -1.571" /> -->
         <parent link="base_link" />
         <child link="sway_stern_thruster_link" />

Commit message: New tuning and hardware physics changes (#3)
* helm config corrections

* new pid values

File: race2_description/urdf/base.urdf.xacro (robot description, xacro)
@@ -64,5 +64,6 @@
     <link name="surge_port_duct_link" />
     <joint name="surge_port_servo_joint" type="fixed">
-        <origin xyz="-0.34 0.079 0.05485" rpy="-1.5707 -1.78 0.52" />
+        <!-- <origin xyz="-0.34 0.079 0.05485" rpy="-1.5707 -1.78 0.52" /> -->
+         <origin xyz="-0.34 0.079 0.05485" rpy="-1.5707 -0.21 0.52" />
         <parent link="base_link" />
         <child link="surge_port_servo_link" />
@@ -73,5 +74,5 @@
         <child link="surge_port_duct_link" />
         <axis xyz="0 0 1" />
-        <limit effort="10" lower="-3.0" upper="3.0" velocity="20" />
+        <limit effort="10" lower="-3.10000000000000" upper="3.10000000000000" velocity="20" />
     </joint>
     <joint name="surge_port_thruster_joint" type="fixed">
@@ -86,5 +87,6 @@
     <link name="surge_starboard_duct_link" />
     <joint name="surge_starboard_servo_joint" type="fixed">
-        <origin xyz="-0.34 -0.079 0.05485" rpy="1.5707 1.78 -0.52" />
+        <!-- <origin xyz="-0.34 -0.079 0.05485" rpy="1.5707 1.78 -0.52" /> -->
+         <origin xyz="-0.34 -0.079 0.05485" rpy="1.5707 0.21 -0.52" />
         <parent link="base_link" />
         <child link="surge_starboard_servo_link" />
@@ -95,5 +97,5 @@
         <child link="surge_starboard_duct_link" />
         <axis xyz="0 0 1" />
-        <limit effort="10" lower="-3.0" upper="3.0" velocity="20" />
+        <limit effort="10" lower="-3.10000000000000" upper="3.10000000000000" velocity="20" />
     </joint>
     <joint name="surge_starboard_thruster_joint" type="fixed">
@@ -149,5 +151,6 @@
     <link name="sway_stern_thruster_link" />
     <joint name="sway_stern_thruster_joint" type="fixed">
-        <origin xyz="-0.216 0.0 0.07535" rpy="3.1415926 0.0 -1.571" />
+        <origin xyz="-0.216 0.0 -0.07535" rpy="3.1415926 0.0 -1.571" />
+        <!-- <origin xyz="-0.216 0.0 0.0" rpy="3.1415926 0.0 -1.571" /> -->
         <parent link="base_link" />
         <child link="sway_stern_thruster_link" />

Commit message: new pid values

File: race2_description/urdf/base.urdf.xacro (robot description, xacro)
@@ -74,5 +74,5 @@
         <child link="surge_port_duct_link" />
         <axis xyz="0 0 1" />
-        <limit effort="10" lower="-3.10000000000000" upper="3.10000000000000" velocity="20" />
+        <limit effort="10" lower="-1.5700000000" upper="1.5700000000" velocity="20" />
     </joint>
     <joint name="surge_port_thruster_joint" type="fixed">
@@ -97,5 +97,5 @@
         <child link="surge_starboard_duct_link" />
         <axis xyz="0 0 1" />
-        <limit effort="10" lower="-3.10000000000000" upper="3.10000000000000" velocity="20" />
+        <limit effort="10" lower="-1.57000000000" upper="1.5700000000" velocity="20" />
     </joint>
     <joint name="surge_starboard_thruster_joint" type="fixed">
@@ -151,6 +151,6 @@
     <link name="sway_stern_thruster_link" />
     <joint name="sway_stern_thruster_joint" type="fixed">
-        <origin xyz="-0.216 0.0 -0.07535" rpy="3.1415926 0.0 -1.571" />
-        <!-- <origin xyz="-0.216 0.0 0.0" rpy="3.1415926 0.0 -1.571" /> -->
+        <!-- <origin xyz="-0.216 0.0 -0.07535" rpy="3.1415926 0.0 -1.571" /> -->
+        <origin xyz="-0.216 0.0 0.0" rpy="3.1415926 0.0 -1.571" />
         <parent link="base_link" />
         <child link="sway_stern_thruster_link" />
