Commit message: added servo joints and tested

File: race2_auv_description/urdf/base.urdf (robot description, URDF)
Before this commit: robot race2_auv, 11 links, 10 joints
Links:
- added link surge_port_thruster_link
- added link surge_starboard_thruster_link
Joints:
- added joint race2_auv/surge_port_servo_joint: type revolute, parent cg_link, child surge_port_thruster_link, origin xyz=-0.86 -0.125 -0.05485 rpy=1.571 0.0 -0.52, axis 0 0 1, limit lower=-1.57100 upper=1.57100 effort=10 velocity=20
- added joint race2_auv/surge_starboard_servo_joint: type revolute, parent cg_link, child surge_starboard_thruster_link, origin xyz=-0.86 0.125 -0.05485 rpy=-1.571 0.0 0.52, axis 0 0 1, limit lower=-1.57100 upper=1.57100 effort=10 velocity=20
- joint base_link: origin xyz=-0.456 0.0 0.0 rpy=0.0 0.0 0.0 -> xyz=-0.0 0.0 0.0 rpy=0.0 0.0 0.0
- joint heave_bow_thruster_joint: origin xyz=-0.07535 0.0 0.07535 rpy=0.0 -1.5707 0.0 -> xyz=-0.07535 0.0 0.07535 rpy=0.0 1.5707 0.0
- joint sway_thruster_joint: origin xyz=0.66635 0.0 0.07535 rpy=0.0 0.0 1.5707 -> xyz=-0.66635 0.0 0.07535 rpy=0.0 0.0 -1.5707

Commit message: testing mvp_control

File: race2_auv_description/urdf/base.urdf (robot description, URDF)
Before this commit: robot race2_auv, 13 links, 12 joints
Joints:
- joint race2_auv/surge_port_servo_joint: limit lower=-1.57100 upper=1.57100 effort=10 velocity=20 -> lower=-3.14 upper=3.14 effort=10 velocity=20
- joint race2_auv/surge_starboard_servo_joint: limit lower=-1.57100 upper=1.57100 effort=10 velocity=20 -> lower=-3.14 upper=3.14 effort=10 velocity=20

Commit message: updated config

File: race2_auv_description/urdf/base.urdf (robot description, URDF)
Before this commit: robot race2_auv, 13 links, 12 joints
Joints:
- joint cg_joint: origin xyz=0.0 0.0 0.0 rpy=3.1415926 0.0 0.0 -> xyz=-0.4 0.0 0.0 rpy=3.1415926 0.0 0.0
- joint race2_auv/surge_port_servo_joint: origin xyz=-0.86 -0.125 -0.05485 rpy=1.571 0.0 -0.52 -> xyz=-0.46 -0.125 -0.05485 rpy=1.571 0.0 -0.52
- joint race2_auv/surge_starboard_servo_joint: origin xyz=-0.86 0.125 -0.05485 rpy=-1.571 0.0 0.52 -> xyz=-0.46 0.125 -0.05485 rpy=-1.571 0.0 0.52

Commit message: added heave stern and correted dvl bug

File: race2_auv_description/urdf/base.urdf (robot description, URDF)
Before this commit: robot race2_auv, 13 links, 12 joints
Links:
- removed link sway_thruster_link
- added link heave_stern_thruster_link
Joints:
- removed joint sway_thruster_joint
- added joint heave_stern_thruster_joint: type fixed, parent base_link, child heave_stern_thruster_link, origin xyz=-0.26635 0.0 0.07535 rpy=0.0 1.5707 0.0
- joint cg_joint: origin xyz=-0.4 0.0 0.0 rpy=3.1415926 0.0 0.0 -> xyz=0.0 0.0 0.0 rpy=3.1415926 0.0 0.0
- joint dvl_joint: origin xyz=-0.5 0.0 0.0 rpy=3.1415926 0.0 0.0 -> xyz=-0.1 0.0 0.0 rpy=3.1415926 0.0 0.0
- joint dvl_sf_joint: origin xyz=-0.5 0.0 0.0 rpy=0.0 0.0 0.0 -> xyz=-0.1 0.0 0.0 rpy=0.0 0.0 0.0
- joint gps_joint: origin xyz=-0.35 0.0 0.4 rpy=0.0 0.0 0.0 -> xyz=0.05 0.0 0.4 rpy=0.0 0.0 0.0
- joint heave_bow_thruster_joint: origin xyz=-0.07535 0.0 0.07535 rpy=0.0 1.5707 0.0 -> xyz=0.32465 0.0 0.07535 rpy=0.0 1.5707 0.0
- joint imu__sf_joint: origin xyz=-0.4 0.0 0.1 rpy=0.0 0.0 0.0 -> xyz=0.0 0.0 0.1 rpy=0.0 0.0 0.0
- joint imu_joint: origin xyz=-0.4 -0.0 0.1 rpy=0.0 0.0 0.0 -> xyz=0.0 -0.0 0.1 rpy=0.0 0.0 0.0
- joint pressure_joint: origin xyz=-0.7 0.0 0.0 rpy=0.0 0.0 0.0 -> xyz=-0.3 0.0 0.0 rpy=0.0 0.0 0.0

Commit message: revert the sway thruster

File: race2_auv_description/urdf/base.urdf (robot description, URDF)
Before this commit: robot race2_auv, 13 links, 12 joints
Links:
- removed link heave_stern_thruster_link
- added link sway_thruster_link
Joints:
- removed joint heave_stern_thruster_joint
- added joint sway_thruster_joint: type fixed, parent base_link, child sway_thruster_link, origin xyz=-0.26635 0.0 0.07535 rpy=0.0 0.0 -1.5707

Commit message: race2 thruster config change

File: race2_auv_description/urdf/base.urdf (robot description, URDF)
Before this commit: robot race2_auv, 13 links, 12 joints
Links:
- removed link sway_thruster_link
- added link heave_stern_thruster_link
Joints:
- removed joint sway_thruster_joint
- added joint heave_stern_thruster_joint: type fixed, parent base_link, child heave_stern_thruster_link, origin xyz=-0.26635 0.0 0.07535 rpy=0.0 1.5707 0.0

Commit message: added two more vector thrusters

File: race2_auv_description/urdf/base.urdf (robot description, URDF)
Before this commit: robot race2_auv, 13 links, 12 joints
Links:
- added link mid_port_thruster_link
- added link mid_starboard_thruster_link
Joints:
- added joint race2_auv/mid_port_servo_joint: type revolute, parent cg_link, child mid_port_thruster_link, origin xyz=-0.06 -0.24 -0.05485 rpy=1.571 0.0 -0.0, axis 0 0 1, limit lower=-3.14 upper=3.14 effort=10 velocity=20
- added joint race2_auv/mid_starboard_servo_joint: type revolute, parent cg_link, child mid_starboard_thruster_link, origin xyz=-0.06 0.24 -0.05485 rpy=-1.571 0.0 0.0, axis 0 0 1, limit lower=-3.14 upper=3.14 effort=10 velocity=20

Commit message: added restoring effort

File: race2_auv_description/urdf/base.urdf (robot description, URDF)
Before this commit: robot race2_auv, 15 links, 14 joints
Links:
- removed link mid_port_thruster_link
- removed link mid_starboard_thruster_link
- added link cb_link
Joints:
- removed joint race2_auv/mid_port_servo_joint
- removed joint race2_auv/mid_starboard_servo_joint
- added joint cb_joint: type fixed, parent base_link, child cb_link, origin xyz=0.0 0.0 0.02 rpy=3.1415926 0.0 0.0
